Commit message: Create a full URDF file for Ufactory Xarm7

File: urdf/ufactory_xarm7.urdf (robot description, URDF)
Before this commit: robot xarm7, 1 links, 0 joints
Links:
- removed link ground_link
- added link base_link; visual mesh filename=package://ufactory_xarm7_description/meshes/link_base.stl scale=1.0 1.0 1.0
- added link gripper; visual mesh filename=package://ufactory_xarm7_description/meshes/gripper_lite.stl scale=1.0 1.0 1.0
- added link link1; visual mesh filename=package://ufactory_xarm7_description/meshes/link1.stl scale=1.0 1.0 1.0
- added link link2; visual mesh filename=package://ufactory_xarm7_description/meshes/link2.stl scale=1.0 1.0 1.0
- added link link3; visual mesh filename=package://ufactory_xarm7_description/meshes/link3.stl scale=1.0 1.0 1.0
- added link link4; visual mesh filename=package://ufactory_xarm7_description/meshes/link4.stl scale=1.0 1.0 1.0
- added link link5; visual mesh filename=package://ufactory_xarm7_description/meshes/link5.stl scale=1.0 1.0 1.0
- added link link6; visual mesh filename=package://ufactory_xarm7_description/meshes/link6.stl scale=1.0 1.0 1.0
- added link link7; visual mesh filename=package://ufactory_xarm7_description/meshes/link7.stl scale=1.0 1.0 1.0
Joints:
- added joint base_link_to_link1: type fixed, parent base_link, child link1, origin xyz=0 0 0.25 rpy=0.0 0.0 0.0
- added joint link1_to_link2: type revolute, parent link1, child link2, origin xyz=0 0 0 rpy=1.57 3.1416 3.1416, axis 0 1 0, limit lower=-6.283 upper=6.283 effort=3.0 velocity=3.14
- added joint link2_to_link3: type revolute, parent link2, child link3, origin xyz=0.05 -0.25 0 rpy=0.0 0.0 3.1416, axis 0 1 0, limit lower=-2.059 upper=2.094 effort=3.0 velocity=3.14
- added joint link3_to_link4: type revolute, parent link3, child link4, origin xyz=0 0 -0.03 rpy=0.0 3.1416 0.0, axis 0 1 0, limit lower=-6.283 upper=6.283 effort=3.0 velocity=3.14
- added joint link4_to_link5: type revolute, parent link4, child link5, origin xyz=0.077 -0.33 0 rpy=1.57 0.0 0.0, axis 0 1 0, limit lower=-0.192 upper=3.927 effort=3.0 velocity=3.14
- added joint link5_to_link6: type revolute, parent link5, child link6, origin xyz=0 0 0 rpy=1.57 0.0 0.0, axis 0 1 0, limit lower=-6.283 upper=6.283 effort=3.0 velocity=3.14
- added joint link6_to_link7: type revolute, parent link6, child link7, axis 0 1 0, limit lower=-1.692 upper=3.142 effort=3.0 velocity=3.14
- added joint link7_to_gripper: type revolute, parent link7, child gripper, origin xyz=0 0 0 rpy=0.0 0.0 0.0, axis 0 1 0, limit lower=-6.283 upper=6.283 effort=3.0 velocity=3.14

Commit message: Change material colour and optimise links orientation

File: urdf/ufactory_xarm7.urdf (robot description, URDF)
Before this commit: robot xarm7, 9 links, 8 joints
Joints:
- joint base_link_to_link1: axis (none) -> 0 1 0; limit (none) -> lower=-6.283 upper=6.283 effort=3.0 velocity=3.14; origin xyz=0 0 0.25 rpy=0.0 0.0 0.0 -> xyz=0 0 0 rpy=0.0 0.0 0.0; type fixed -> revolute
- joint link1_to_link2: limit lower=-6.283 upper=6.283 effort=3.0 velocity=3.14 -> lower=-2.059 upper=2.094 effort=3.0 velocity=3.14; origin xyz=0 0 0 rpy=1.57 3.1416 3.1416 -> xyz=0 0 0 rpy=0.0 0.0 0.0
- joint link2_to_link3: limit lower=-2.059 upper=2.094 effort=3.0 velocity=3.14 -> lower=-6.283 upper=6.283 effort=3.0 velocity=3.14; origin xyz=0.05 -0.25 0 rpy=0.0 0.0 3.1416 -> xyz=0 0 0 rpy=0.0 0.0 0.0
- joint link3_to_link4: limit lower=-6.283 upper=6.283 effort=3.0 velocity=3.14 -> lower=-0.192 upper=3.927 effort=3.0 velocity=3.14; origin xyz=0 0 -0.03 rpy=0.0 3.1416 0.0 -> xyz=0 0 0 rpy=0.0 0.0 0.0
- joint link4_to_link5: limit lower=-0.192 upper=3.927 effort=3.0 velocity=3.14 -> lower=-6.283 upper=6.283 effort=3.0 velocity=3.14; origin xyz=0.077 -0.33 0 rpy=1.57 0.0 0.0 -> xyz=0 0 0 rpy=0.0 0.0 0.0
- joint link5_to_link6: limit lower=-6.283 upper=6.283 effort=3.0 velocity=3.14 -> lower=-1.692 upper=3.142 effort=3.0 velocity=3.14; origin xyz=0 0 0 rpy=1.57 0.0 0.0 -> xyz=0 0 0 rpy=0.0 0.0 0.0
- joint link6_to_link7: limit lower=-1.692 upper=3.142 effort=3.0 velocity=3.14 -> lower=-6.283 upper=6.283 effort=3.0 velocity=3.14; origin (none) -> xyz=0 0 0 rpy=0.0 0.0 0.0
- joint link7_to_gripper: axis 0 1 0 -> (none); limit lower=-6.283 upper=6.283 effort=3.0 velocity=3.14 -> (none); type revolute -> fixed

Commit message: update origin

File: urdf/ufactory_xarm7.urdf (robot description, URDF)
Before this commit: robot xarm7, 9 links, 8 joints
Joints:
- joint base_link_to_link1: origin xyz=0 0 0 rpy=0.0 0.0 0.0 -> xyz=0 0 0.25 rpy=0.0 0.0 0.0
- joint link1_to_link2: origin xyz=0 0 0 rpy=0.0 0.0 0.0 -> xyz=0 0 0 rpy=1.57 3.1416 3.1416
- joint link2_to_link3: origin xyz=0 0 0 rpy=0.0 0.0 0.0 -> xyz=0.05 -0.25 0 rpy=0.0 0.0 3.1416
- joint link3_to_link4: origin xyz=0 0 0 rpy=0.0 0.0 0.0 -> xyz=0 0 -0.03 rpy=0.0 3.1416 0.0
- joint link4_to_link5: origin xyz=0 0 0 rpy=0.0 0.0 0.0 -> xyz=0.077 -0.33 0 rpy=1.57 0.0 0.0
- joint link5_to_link6: origin xyz=0 0 0 rpy=0.0 0.0 0.0 -> xyz=0 0 0 rpy=1.57 0.0 0.0
- joint link7_to_gripper: origin xyz=0 0 0 rpy=0.0 0.0 0.0 -> xyz=0.077 0.0605 0.0 rpy=-1.571 1.571 0.0
