Commit message: Create Xacro model and auto-generate URDF

File: urdf/joints.xacro (robot description, xacro)
@@ -21,7 +21,7 @@
                     lower="-1.692" upper="3.142"/>
   <xacro:u_xarm7_joint name="link6_to_link7" parent="link6" child="link7"
-                    xyz="0.0 0.0 0.0" rpy="0.0 0.0 0.0" axis="0 1 0"
+                    xyz="0.078 0.065 0.0" rpy="1.57 0.0 0.0" axis="0 1 0"
                     lower="-6.283" upper="6.283"/>
   <xacro:u_xarm7_fixed name="link7_to_gripper" parent="link7" child="gripper"
-                    xyz="0.077 0.0605 0.0" rpy="-1.571 1.571 0.0"/>
+                    xyz="0.0 0.0 -0.025" rpy="0.0 3.141 1.571"/>
 </robot>

File: urdf/macros.xacro (robot description, xacro)
@@ -11,4 +11,10 @@
         <material name="white"/>
       </visual>
+      <collision>
+        <origin xyz="0 0 0" rpy="0 0 0"/>
+        <geometry>
+          <mesh filename="package://ufactory_xarm7_description/meshes/${mesh}" scale="1.0 1.0 1.0"/>
+        </geometry>
+      </collision>
     </link>
   </xacro:macro>

File: urdf/ufactory_xarm7.urdf (robot description, URDF)
Before this commit: robot xarm7, 9 links, 8 joints
Joints:
- joint link6_to_link7: origin xyz=0 0 0 rpy=0.0 0.0 0.0 -> xyz=0.078 0.065 0.0 rpy=1.57 0.0 0.0
- joint link7_to_gripper: origin xyz=0.077 0.0605 0.0 rpy=-1.571 1.571 0.0 -> xyz=0.0 0.0 -0.025 rpy=0.0 3.141 1.571

File: urdf/xarm7.urdf (robot description, URDF)
Before this commit: robot ufactory-xarm7-robot, 9 links, 8 joints
Links:
- link base_link: geometry collision mesh filename=package://ufactory_xarm7_description/meshes/link_base.stl scale=1.0 1.0 1.0; visual mesh filename=package://ufactory_xarm7_description/meshes/link_base.stl scale=1.0 1.0 1.0
- link gripper: geometry collision mesh filename=package://ufactory_xarm7_description/meshes/gripper_lite.stl scale=1.0 1.0 1.0; visual mesh filename=package://ufactory_xarm7_description/meshes/gripper_lite.stl scale=1.0 1.0 1.0
- link link1: geometry collision mesh filename=package://ufactory_xarm7_description/meshes/link1.stl scale=1.0 1.0 1.0; visual mesh filename=package://ufactory_xarm7_description/meshes/link1.stl scale=1.0 1.0 1.0
- link link2: geometry collision mesh filename=package://ufactory_xarm7_description/meshes/link2.stl scale=1.0 1.0 1.0; visual mesh filename=package://ufactory_xarm7_description/meshes/link2.stl scale=1.0 1.0 1.0
- link link3: geometry collision mesh filename=package://ufactory_xarm7_description/meshes/link3.stl scale=1.0 1.0 1.0; visual mesh filename=package://ufactory_xarm7_description/meshes/link3.stl scale=1.0 1.0 1.0
- link link4: geometry collision mesh filename=package://ufactory_xarm7_description/meshes/link4.stl scale=1.0 1.0 1.0; visual mesh filename=package://ufactory_xarm7_description/meshes/link4.stl scale=1.0 1.0 1.0
- link link5: geometry collision mesh filename=package://ufactory_xarm7_description/meshes/link5.stl scale=1.0 1.0 1.0; visual mesh filename=package://ufactory_xarm7_description/meshes/link5.stl scale=1.0 1.0 1.0
- link link6: geometry collision mesh filename=package://ufactory_xarm7_description/meshes/link6.stl scale=1.0 1.0 1.0; visual mesh filename=package://ufactory_xarm7_description/meshes/link6.stl scale=1.0 1.0 1.0
- link link7: geometry collision mesh filename=package://ufactory_xarm7_description/meshes/link7.stl scale=1.0 1.0 1.0; visual mesh filename=package://ufactory_xarm7_description/meshes/link7.stl scale=1.0 1.0 1.0
Joints:
- joint link6_to_link7: origin xyz=0.0 0.0 0.0 rpy=0.0 0.0 0.0 -> xyz=0.078 0.065 0.0 rpy=1.57 0.0 0.0
- joint link7_to_gripper: origin xyz=0.077 0.0605 0.0 rpy=-1.571 1.571 0.0 -> xyz=0.0 0.0 -0.025 rpy=0.0 3.141 1.571

File: urdf/xarm7.urdf.xacro (robot description, xacro)
@@ -6,4 +6,5 @@
   <xacro:include filename="macros.xacro"/>
   <xacro:include filename="joints.xacro"/>
+  <xacro:property name="gazebo_control" value="flase" />
   <!-- Load robot color -->
   <xacro:material_white/>
