Commit message: Fix collision issue

File: ufactory_xarm7_description/urdf/macros.xacro (robot description, xacro)
@@ -11,4 +11,10 @@
         <material name="white"/>
       </visual>
+      <collision>
+        <origin xyz="0 0 0" rpy="0 0 0"/>
+        <geometry>
+          <mesh filename="package://ufactory_xarm7_description/meshes/${mesh}" scale="1.0 1.0 1.0"/>
+        </geometry>
+      </collision>
     </link>
   </xacro:macro>

File: ufactory_xarm7_description/urdf/xarm7.urdf (robot description, URDF)
Before this commit: robot ufactory-xarm7-robot, 9 links, 8 joints
Links:
- link base_link: geometry collision mesh filename=package://ufactory_xarm7_description/meshes/link_base.stl scale=1.0 1.0 1.0; visual mesh filename=package://ufactory_xarm7_description/meshes/link_base.stl scale=1.0 1.0 1.0
- link gripper: geometry collision mesh filename=package://ufactory_xarm7_description/meshes/gripper_lite.stl scale=1.0 1.0 1.0; visual mesh filename=package://ufactory_xarm7_description/meshes/gripper_lite.stl scale=1.0 1.0 1.0
- link link1: geometry collision mesh filename=package://ufactory_xarm7_description/meshes/link1.stl scale=1.0 1.0 1.0; visual mesh filename=package://ufactory_xarm7_description/meshes/link1.stl scale=1.0 1.0 1.0
- link link2: geometry collision mesh filename=package://ufactory_xarm7_description/meshes/link2.stl scale=1.0 1.0 1.0; visual mesh filename=package://ufactory_xarm7_description/meshes/link2.stl scale=1.0 1.0 1.0
- link link3: geometry collision mesh filename=package://ufactory_xarm7_description/meshes/link3.stl scale=1.0 1.0 1.0; visual mesh filename=package://ufactory_xarm7_description/meshes/link3.stl scale=1.0 1.0 1.0
- link link4: geometry collision mesh filename=package://ufactory_xarm7_description/meshes/link4.stl scale=1.0 1.0 1.0; visual mesh filename=package://ufactory_xarm7_description/meshes/link4.stl scale=1.0 1.0 1.0
- link link5: geometry collision mesh filename=package://ufactory_xarm7_description/meshes/link5.stl scale=1.0 1.0 1.0; visual mesh filename=package://ufactory_xarm7_description/meshes/link5.stl scale=1.0 1.0 1.0
- link link6: geometry collision mesh filename=package://ufactory_xarm7_description/meshes/link6.stl scale=1.0 1.0 1.0; visual mesh filename=package://ufactory_xarm7_description/meshes/link6.stl scale=1.0 1.0 1.0
- link link7: geometry collision mesh filename=package://ufactory_xarm7_description/meshes/link7.stl scale=1.0 1.0 1.0; visual mesh filename=package://ufactory_xarm7_description/meshes/link7.stl scale=1.0 1.0 1.0

File: ufactory_xarm7_description/urdf/xarm7.urdf.xacro (robot description, xacro)
@@ -6,4 +6,5 @@
   <xacro:include filename="macros.xacro"/>
   <xacro:include filename="joints.xacro"/>
+  <xacro:property name="gazebo_control" value="false" />
   <!-- Load robot color -->
   <xacro:material_white/>
