Commit message: Redefine joints and links

File: ufactory_xarm7_description/urdf/joints.xacro (robot description, xacro)
@@ -3,25 +3,25 @@
   <!-- Define joints -->
   <xacro:u_xarm7_joint name="base_link_to_link1" parent="base_link" child="link1"
-                    xyz="0 0 0.25" rpy="0.0 0.0 0.0" axis="0 1 0"
+                    xyz="0.0 0.0 0.15" rpy="0.0 0.0 0.0" axis="0 1 0"
                     lower="-6.283" upper="6.283"/>
   <xacro:u_xarm7_joint name="link1_to_link2" parent="link1" child="link2"
-                    xyz="0 0 0" rpy="1.57 3.1416 3.1416" axis="0 1 0"
+                    xyz="0.0 0.077 0.11" rpy="0.0 0.0 0.0" axis="0 1 0"
                     lower="-2.059" upper="2.094"/>
   <xacro:u_xarm7_joint name="link2_to_link3" parent="link2" child="link3"
-                    xyz="0.05 -0.25 0" rpy="0.0 0.0 3.1416" axis="0 1 0"
+                    xyz="0.0 -0.075 0.18" rpy="0.0 0.0 0.0" axis="0 1 0"
                     lower="-6.283" upper="6.283"/>
   <xacro:u_xarm7_joint name="link3_to_link4" parent="link3" child="link4"
-                    xyz="0.0 0.0 -0.03" rpy="0.0 3.1416 0.0" axis="0 1 0"
+                    xyz="0.055 -0.055 0.099" rpy="0.0 0.0 0.0" axis="0 1 0"
                     lower="-0.192" upper="3.927"/>
   <xacro:u_xarm7_joint name="link4_to_link5" parent="link4" child="link5"
-                    xyz="0.077 -0.33 0" rpy="1.57 0.0 0.0" axis="0 1 0"
+                    xyz="0.078 0.058 -0.16" rpy="0.0 0.0 0.0" axis="0 1 0"
                     lower="-6.283" upper="6.283"/>
   <xacro:u_xarm7_joint name="link5_to_link6" parent="link5" child="link6"
-                    xyz="0 0 0" rpy="1.57 0.0 0.0" axis="0 1 0"
+                    xyz="0.0 0.0 -0.17" rpy="0.0 0.0 0.0" axis="0 1 0"
                     lower="-1.692" upper="3.142"/>
   <xacro:u_xarm7_joint name="link6_to_link7" parent="link6" child="link7"
-                    xyz="0.0 0.0 0.0" rpy="0.0 0.0 0.0" axis="0 1 0"
+                    xyz="0.072 0.0 -0.072" rpy="0.0 0.0 0.0" axis="0 1 0"
                     lower="-6.283" upper="6.283"/>
   <xacro:u_xarm7_fixed name="link7_to_gripper" parent="link7" child="gripper"
-                    xyz="0.077 0.0605 0.0" rpy="-1.571 1.571 0.0"/>
+                    xyz="0.0 0.0 -0.02" rpy="0.0 0.0 0.0"/>
 </robot>

File: ufactory_xarm7_description/urdf/macros.xacro (robot description, xacro)
@@ -2,21 +2,21 @@
 <robot xmlns:xacro="http://ros.org/wiki/xacro">
   <!-- Set Link macro -->
-  <xacro:macro name="u_xarm7_link" params="name mesh">
-    <link name="${name}">
-      <visual>
-        <origin xyz="0 0 0" rpy="0 0 0"/>
-        <geometry>
-          <mesh filename="package://ufactory_xarm7_description/meshes/${mesh}" scale="1.0 1.0 1.0"/>
-        </geometry>
-        <material name="white"/>
-      </visual>
-      <collision>
-        <origin xyz="0 0 0" rpy="0 0 0"/>
-        <geometry>
-          <mesh filename="package://ufactory_xarm7_description/meshes/${mesh}" scale="1.0 1.0 1.0"/>
-        </geometry>
-      </collision>
-    </link>
-  </xacro:macro>
+<xacro:macro name="u_xarm7_link" params="name mesh xyz rpy">
+  <link name="${name}">
+    <visual>
+      <origin xyz="${xyz}" rpy="${rpy}"/>
+      <geometry>
+        <mesh filename="package://ufactory_xarm7_description/meshes/${mesh}"/>
+      </geometry>
+      <material name="white"/>
+    </visual>
+    <collision>
+      <origin xyz="${xyz}" rpy="${rpy}"/>
+      <geometry>
+        <mesh filename="package://ufactory_xarm7_description/meshes/${mesh}"/>
+      </geometry>
+    </collision>
+  </link>
+</xacro:macro>
   <!-- Define revolute joint macro -->
   <xacro:macro name="u_xarm7_joint" params="name parent child xyz rpy axis lower upper">

File: ufactory_xarm7_description/urdf/xarm7.urdf (robot description, URDF)
Before this commit: robot ufactory-xarm7-robot, 9 links, 8 joints
Links:
- link base_link: geometry collision mesh filename=package://ufactory_xarm7_description/meshes/link_base.stl; visual mesh filename=package://ufactory_xarm7_description/meshes/link_base.stl
- link gripper: geometry collision mesh filename=package://ufactory_xarm7_description/meshes/gripper_lite.stl; visual mesh filename=package://ufactory_xarm7_description/meshes/gripper_lite.stl
- link link1: geometry collision mesh filename=package://ufactory_xarm7_description/meshes/link1.stl; visual mesh filename=package://ufactory_xarm7_description/meshes/link1.stl
- link link2: geometry collision mesh filename=package://ufactory_xarm7_description/meshes/link2.stl; visual mesh filename=package://ufactory_xarm7_description/meshes/link2.stl
- link link3: geometry collision mesh filename=package://ufactory_xarm7_description/meshes/link3.stl; visual mesh filename=package://ufactory_xarm7_description/meshes/link3.stl
- link link4: geometry collision mesh filename=package://ufactory_xarm7_description/meshes/link4.stl; visual mesh filename=package://ufactory_xarm7_description/meshes/link4.stl
- link link5: geometry collision mesh filename=package://ufactory_xarm7_description/meshes/link5.stl; visual mesh filename=package://ufactory_xarm7_description/meshes/link5.stl
- link link6: geometry collision mesh filename=package://ufactory_xarm7_description/meshes/link6.stl; visual mesh filename=package://ufactory_xarm7_description/meshes/link6.stl
- link link7: geometry collision mesh filename=package://ufactory_xarm7_description/meshes/link7.stl; visual mesh filename=package://ufactory_xarm7_description/meshes/link7.stl
Joints:
- joint base_link_to_link1: origin xyz=0 0 0.25 rpy=0.0 0.0 0.0 -> xyz=0.0 0.0 0.15 rpy=0.0 0.0 0.0
- joint link1_to_link2: origin xyz=0 0 0 rpy=1.57 3.1416 3.1416 -> xyz=0.0 0.077 0.11 rpy=0.0 0.0 0.0
- joint link2_to_link3: origin xyz=0.05 -0.25 0 rpy=0.0 0.0 3.1416 -> xyz=0.0 -0.075 0.18 rpy=0.0 0.0 0.0
- joint link3_to_link4: origin xyz=0.0 0.0 -0.03 rpy=0.0 3.1416 0.0 -> xyz=0.055 -0.055 0.099 rpy=0.0 0.0 0.0
- joint link4_to_link5: origin xyz=0.077 -0.33 0 rpy=1.57 0.0 0.0 -> xyz=0.078 0.058 -0.16 rpy=0.0 0.0 0.0
- joint link5_to_link6: origin xyz=0 0 0 rpy=1.57 0.0 0.0 -> xyz=0.0 0.0 -0.17 rpy=0.0 0.0 0.0
- joint link6_to_link7: origin xyz=0.0 0.0 0.0 rpy=0.0 0.0 0.0 -> xyz=0.072 0.0 -0.072 rpy=0.0 0.0 0.0
- joint link7_to_gripper: origin xyz=0.077 0.0605 0.0 rpy=-1.571 1.571 0.0 -> xyz=0.0 0.0 -0.02 rpy=0.0 0.0 0.0

File: ufactory_xarm7_description/urdf/xarm7.urdf.xacro (robot description, xacro)
@@ -6,16 +6,7 @@
   <xacro:include filename="macros.xacro"/>
   <xacro:include filename="joints.xacro"/>
+  <xacro:include filename="links.xacro"/>
   <xacro:property name="gazebo_control" value="false" />
   <!-- Load robot color -->
   <xacro:material_white/>
-  <!-- Define links -->
-  <xacro:u_xarm7_link name="base_link" mesh="link_base.stl"/>
-  <xacro:u_xarm7_link name="link1" mesh="link1.stl"/>
-  <xacro:u_xarm7_link name="link2" mesh="link2.stl"/>
-  <xacro:u_xarm7_link name="link3" mesh="link3.stl"/>
-  <xacro:u_xarm7_link name="link4" mesh="link4.stl"/>
-  <xacro:u_xarm7_link name="link5" mesh="link5.stl"/>
-  <xacro:u_xarm7_link name="link6" mesh="link6.stl"/>
-  <xacro:u_xarm7_link name="link7" mesh="link7.stl"/>
-  <xacro:u_xarm7_link name="gripper" mesh="gripper_lite.stl"/>
 </robot>
